File: nixie-tube-clock-hw/12_150_Boost.kicad_sch (KiCad schematic)
At the start: 35 parts, among them Q1 FQD16N25CTM, Q2 PMBT3906,235, U1 MC34063AD, U2 AS321KTR-G1

Commit message: 1
Parts:
- TP1, TP2, TP3, TP4: footprint TestPoint:TestPoint_Pad_D1.5mm -> TestPoint:TestPoint_Pad_D3.0mm
- TP5: footprint TestPoint:TestPoint_Keystone_5000-5004_Miniature -> TestPoint:TestPoint_Pad_D3.0mm
Changed lines of the file:
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@@
       (effects (font (size 1.27 1.27)) (justify left) hide)
     )
-    (property "Footprint" "TestPoint:TestPoint_Pad_D1.5mm" (id 2) (at 68.58 53.34 0)
+    (property "Footprint" "TestPoint:TestPoint_Pad_D3.0mm" (id 2) (at 68.58 53.34 0)
       (effects (font (size 1.27 1.27)) hide)
     )
@@
       (effects (font (size 1.27 1.27)) (justify left) hide)
     )
-    (property "Footprint" "TestPoint:TestPoint_Keystone_5000-5004_Miniature" (id 2) (at 233.68 95.25 0)
+    (property "Footprint" "TestPoint:TestPoint_Pad_D3.0mm" (id 2) (at 233.68 95.25 0)
       (effects (font (size 1.27 1.27)) hide)
     )
@@
       (effects (font (size 1.27 1.27)) (justify left) hide)
     )
-    (property "Footprint" "TestPoint:TestPoint_Pad_D1.5mm" (id 2) (at 220.98 71.12 0)
+    (property "Footprint" "TestPoint:TestPoint_Pad_D3.0mm" (id 2) (at 220.98 71.12 0)
       (effects (font (size 1.27 1.27)) hide)
     )
@@
       (effects (font (size 1.27 1.27)) (justify left) hide)
     )
-    (property "Footprint" "TestPoint:TestPoint_Pad_D1.5mm" (id 2) (at 220.98 83.82 0)
+    (property "Footprint" "TestPoint:TestPoint_Pad_D3.0mm" (id 2) (at 220.98 83.82 0)
       (effects (font (size 1.27 1.27)) hide)
     )
@@
       (effects (font (size 1.27 1.27)) (justify left) hide)
     )
-    (property "Footprint" "TestPoint:TestPoint_Pad_D1.5mm" (id 2) (at 91.44 53.34 0)
-      (effects (font (size 1.27 1.27)) hide)
-    )
+    (property "Footprint" "TestPoint:TestPoint_Pad_D3.0mm" (id 2) (at 91.44 53.34 0)
+      (effects (font (size 1.27 1.27)) hide)
+    )

Commit message: minor board / part changes
Parts:
- L1: value 1mH -> 470uH
Changed lines of the file:
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@@
       (effects (font (size 1.27 1.27)) (justify left))
     )
-    (property "Value" "1mH" (id 1) (at 129.5908 63.373 0)
+    (property "Value" "470uH" (id 1) (at 129.5908 63.373 0)
       (effects (font (size 1.27 1.27)) (justify left))
     )
@@
       (effects (font (size 1.27 1.27)) hide)
     )
-    (property "Datasheet" "PM2110-102K-RC" (id 3) (at 128.27 62.23 0)
+    (property "Datasheet" "PM2120-471K-RC" (id 3) (at 128.27 62.23 0)
       (effects (font (size 1.27 1.27)) hide)
     )
@@
       (effects (font (size 1.27 1.27)) hide)
     )
-    (property "Datasheet" "RT0805FRE07180KL" (id 3) (at 148.59 95.25 0)
-      (effects (font (size 1.27 1.27)) hide)
-    )
+    (property "Datasheet" "" (id 3) (at 148.59 95.25 0)
+      (effects (font (size 1.27 1.27)) hide)
+    )
