File: nixie-tube-clock-hw/IN12A-Driver.kicad_sch (KiCad schematic)
At the start: 26 parts

Commit message: layout and routing
Parts:
- added J3: LPPB121NFSC-RC, symbol nixie-tube-clock:BOMTIE
- C17, C18: renamed from C?; footprint Capacitor_SMD:C_0603_1608Metric -> Capacitor_SMD:C_0805_2012Metric
- IN-12A_2: renamed from NT?; value IN-12A -> IN-12A DAUGHTER; footprint (none) -> nixie_tube_clock:nixie_daughter
- R44, R45, R46, R48, R49, R50, R51, R52, R53, R54: renamed from R?; footprint Resistor_SMD:R_0603_1608Metric -> Resistor_SMD:R_0805_2012Metric
- U7, U8: renamed from U?; footprint (none) -> Package_SO:SOIC-16_3.9x9.9mm_P1.27mm
- gave numbers to parts that had none: 11

Commit message: 1
Parts:
- renumbered C17 to C21, C18 to C22, IN-12A_2 to IN-12A_4, J3 to J5, Q17 to Q37, Q18 to Q38, Q19 to Q39, Q20 to Q40, Q21 to Q41, Q22 to Q42, Q23 to Q43, Q24 to Q44, Q25 to Q45, Q26 to Q46, R44 to R66, R45 to R67, R46 to R68, R47 to R69, R48 to R70, R49 to R71, R50 to R72, R51 to R73, R52 to R74, R53 to R75, R54 to R76, U7 to U11, U8 to U12

Commit message: a
Parts:
- U5: renamed from U11; value 74HC594D,118 -> (none); footprint Package_SO:SOIC-16_3.9x9.9mm_P1.27mm -> (none)
- U6: renamed from U12; value 74HC594D,118 -> (none); footprint Package_SO:SOIC-16_3.9x9.9mm_P1.27mm -> (none)
- renumbered C21 to C15, C22 to C16, IN-12A_4 to IN-12A_1, J5 to J2, Q40 to Q10, Q41 to Q11, Q42 to Q12, Q43 to Q13, Q44 to Q14, Q45 to Q15, Q46 to Q16, Q37 to Q7, Q38 to Q8, Q39 to Q9, R66 to R33, R67 to R34, R68 to R35, R69 to R36, R70 to R37, R71 to R38, R72 to R39, R73 to R40, R74 to R41, R75 to R42, R76 to R43
