File: nixie-tube-clock-hw/nixie-tube-clock.kicad_sch (KiCad schematic)
At the start: 37 parts, among them J1 PJ-036AH-SMT-TR, Q3 MMSTA42-7-F, Q4 MMSTA42-7-F, Q5 MMSTA42-7-F, Q6 MMSTA42-7-F, U3 ItsyBitsy_M0_Express, U4 NCP1117IDT50T4G

Commit message: 1
Parts:
- added H1, H2, H3, H4, H5, H6, H7, H8: #6, nixie_tube_clock:#6 Hole, symbol Mechanical:MountingHole
Changed lines of the file:
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@@
     (pin "2")
+  )
+  (symbol (lib_id "Mechanical:MountingHole") (at 255.27 133.35 0) (unit 1)
+    (in_bom yes) (on_board yes) (fields_autoplaced)
+    (property "Reference" "H1" (id 0) (at 257.81 132.0799 0)
+      (effects (font (size 1.27 1.27)) (justify left) hide)
+    )
+    (property "Value" "#6" (id 1) (at 257.81 134.6199 0)
+      (effects (font (size 1.27 1.27)) (justify left))
+    )
+    (property "Footprint" "nixie_tube_clock:#6 Hole" (id 2) (at 255.27 133.35 0)
+      (effects (font (size 1.27 1.27)) hide)
+    )
+    (property "Datasheet" "~" (id 3) (at 255.27 133.35 0)
+      (effects (font (size 1.27 1.27)) hide)
+    )
   )
   (symbol (lib_id "Device:R_US") (at 30.48 165.1 90) (unit 1)
@@
     (pin "1")
   )
+  (symbol (lib_id "Mechanical:MountingHole") (at 255.27 143.51 0) (unit 1)
+    (in_bom yes) (on_board yes) (fields_autoplaced)
+    (property "Reference" "H3" (id 0) (at 257.81 142.2399 0)
+      (effects (font (size 1.27 1.27)) (justify left) hide)
+    )
+    (property "Value" "#6" (id 1) (at 257.81 144.7799 0)
+      (effects (font (size 1.27 1.27)) (justify left))
+    )
+    (property "Footprint" "nixie_tube_clock:#6 Hole" (id 2) (at 255.27 143.51 0)
+      (effects (font (size 1.27 1.27)) hide)
+    )
+    (property "Datasheet" "~" (id 3) (at 255.27 143.51 0)
+      (effects (font (size 1.27 1.27)) hide)
+    )
+  )
   (symbol (lib_id "Device:R_US") (at 142.24 67.31 270) (mirror x) (unit 1)
     (in_bom yes) (on_board yes)
@@
     (pin "1")
   )
+  (symbol (lib_id "Mechanical:MountingHole") (at 255.27 148.59 0) (unit 1)
+    (in_bom yes) (on_board yes) (fields_autoplaced)
+    (property "Reference" "H4" (id 0) (at 257.81 147.3199 0)
+      (effects (font (size 1.27 1.27)) (justify left) hide)
+    )
+    (property "Value" "#6" (id 1) (at 257.81 149.8599 0)
+      (effects (font (size 1.27 1.27)) (justify left))
+    )
+    (property "Footprint" "nixie_tube_clock:#6 Hole" (id 2) (at 255.27 148.59 0)
+      (effects (font (size 1.27 1.27)) hide)
+    )
+    (property "Datasheet" "~" (id 3) (at 255.27 148.59 0)
+      (effects (font (size 1.27 1.27)) hide)
+    )
+  )
   (symbol (lib_id "Device:Q_NPN_BEC") (at 109.22 167.64 0) (unit 1)
     (in_bom yes) (on_board yes) (fields_autoplaced)
@@
     (pin "1")
     (pin "2")
+  )
+  (symbol (lib_id "Mechanical:MountingHole") (at 255.27 153.67 0) (unit 1)
+    (in_bom yes) (on_board yes) (fields_autoplaced)
+    (property "Reference" "H5" (id 0) (at 257.81 152.3999 0)
+      (effects (font (size 1.27 1.27)) (justify left) hide)
+    )
+    (property "Value" "#6" (id 1) (at 257.81 154.9399 0)
+      (effects (font (size 1.27 1.27)) (justify left))
+    )
+    (property "Footprint" "nixie_tube_clock:#6 Hole" (id 2) (at 255.27 153.67 0)
+      (effects (font (size 1.27 1.27)) hide)
+    )
+    (property "Datasheet" "~" (id 3) (at 255.27 153.67 0)
+      (effects (font (size 1.27 1.27)) hide)
+    )
   )
   (symbol (lib_id "power:+3.3V") (at 111.76 147.32 0) (mirror y) (unit 1)
@@
     (pin "1")
     (pin "2")
+  )
+  (symbol (lib_id "Mechanical:MountingHole") (at 255.27 158.75 0) (unit 1)
+    (in_bom yes) (on_board yes) (fields_autoplaced)
+    (property "Reference" "H6" (id 0) (at 257.81 157.4799 0)
+      (effects (font (size 1.27 1.27)) (justify left) hide)
+    )
+    (property "Value" "#6" (id 1) (at 257.81 160.0199 0)
+      (effects (font (size 1.27 1.27)) (justify left))
+    )
+    (property "Footprint" "nixie_tube_clock:#6 Hole" (id 2) (at 255.27 158.75 0)
+      (effects (font (size 1.27 1.27)) hide)
+    )
+    (property "Datasheet" "~" (id 3) (at 255.27 158.75 0)
+      (effects (font (size 1.27 1.27)) hide)
+    )
   )
   (symbol (lib_id "power:+3.3V") (at 80.01 36.83 0) (mirror y) (unit 1)
@@
     (pin "1")
   )
+  (symbol (lib_id "Mechanical:MountingHole") (at 265.43 133.35 0) (unit 1)
+    (in_bom yes) (on_board yes) (fields_autoplaced)
+    (property "Reference" "H7" (id 0) (at 267.97 132.0799 0)
+      (effects (font (size 1.27 1.27)) (justify left) hide)
+    )
+    (property "Value" "#6" (id 1) (at 267.97 134.6199 0)
+      (effects (font (size 1.27 1.27)) (justify left))
+    )
+    (property "Footprint" "nixie_tube_clock:#6 Hole" (id 2) (at 265.43 133.35 0)
+      (effects (font (size 1.27 1.27)) hide)
+    )
+    (property "Datasheet" "~" (id 3) (at 265.43 133.35 0)
+      (effects (font (size 1.27 1.27)) hide)
+    )
+  )
   (symbol (lib_id "Device:R_US") (at 142.24 54.61 90) (unit 1)
     (in_bom yes) (on_board yes)
@@
     (pin "2")
   )
+  (symbol (lib_id "Mechanical:MountingHole") (at 265.43 138.43 0) (unit 1)
+    (in_bom yes) (on_board yes) (fields_autoplaced)
+    (property "Reference" "H8" (id 0) (at 267.97 137.1599 0)
+      (effects (font (size 1.27 1.27)) (justify left) hide)
+    )
+    (property "Value" "#6" (id 1) (at 267.97 139.6999 0)
+      (effects (font (size 1.27 1.27)) (justify left))
+    )
+    (property "Footprint" "nixie_tube_clock:#6 Hole" (id 2) (at 265.43 138.43 0)
+      (effects (font (size 1.27 1.27)) hide)
+    )
+    (property "Datasheet" "~" (id 3) (at 265.43 138.43 0)
+      (effects (font (size 1.27 1.27)) hide)
+    )
+  )
   (symbol (lib_id "Device:R_US") (at 104.14 44.45 90) (unit 1)
     (in_bom yes) (on_board yes)
@@
     (pin "1")
     (pin "2")
+  )
+  (symbol (lib_id "Mechanical:MountingHole") (at 255.27 138.43 0) (unit 1)
+    (in_bom yes) (on_board yes) (fields_autoplaced)
+    (property "Reference" "H2" (id 0) (at 257.81 137.1599 0)
+      (effects (font (size 1.27 1.27)) (justify left) hide)
+    )
+    (property "Value" "#6" (id 1) (at 257.81 139.6999 0)
+      (effects (font (size 1.27 1.27)) (justify left))
+    )
+    (property "Footprint" "nixie_tube_clock:#6 Hole" (id 2) (at 255.27 138.43 0)
+      (effects (font (size 1.27 1.27)) hide)
+    )
+    (property "Datasheet" "~" (id 3) (at 255.27 138.43 0)
+      (effects (font (size 1.27 1.27)) hide)
+    )
   )
   (symbol (lib_id "power:GND") (at 149.86 172.72 0) (unit 1)
@@
       (reference "D8") (unit 1) (value "ORANGE") (footprint "Diode_SMD:D_0805_2012Metric")
     )
+    (path "/2db578cd-b125-49d3-b68b-3360b8f58d41"
+      (reference "H1") (unit 1) (value "#6") (footprint "nixie_tube_clock:#6 Hole")
+    )
+    (path "/f21eb6e0-87b3-4845-8fb5-6a09c9a60a2b"
+      (reference "H2") (unit 1) (value "#6") (footprint "nixie_tube_clock:#6 Hole")
+    )
+    (path "/5bc16b3a-a1cd-4002-8881-eefa1f194921"
+      (reference "H3") (unit 1) (value "#6") (footprint "nixie_tube_clock:#6 Hole")
+    )
+    (path "/6c8fe750-f5d5-45e3-8031-75f1034c352b"
+      (reference "H4") (unit 1) (value "#6") (footprint "nixie_tube_clock:#6 Hole")
+    )
+    (path "/7d326b37-ab5e-44d1-b94f-8bb8a3082b83"
+      (reference "H5") (unit 1) (value "#6") (footprint "nixie_tube_clock:#6 Hole")
+    )
+    (path "/a154a455-559c-42cb-8a6a-f9d854eee6d4"
+      (reference "H6") (unit 1) (value "#6") (footprint "nixie_tube_clock:#6 Hole")
+    )
+    (path "/bfc01b44-7156-41e7-98cb-597e08375c1a"
+      (reference "H7") (unit 1) (value "#6") (footprint "nixie_tube_clock:#6 Hole")
+    )
+    (path "/c92a0d2e-9a0b-4896-833d-795750b03fbe"
+      (reference "H8") (unit 1) (value "#6") (footprint "nixie_tube_clock:#6 Hole")
+    )
     (path "/3e56d9ee-e4f1-41fc-9d6a-2d6e6e8ad807/1bcadabf-49fd-4f15-9703-c271281f3d0c"
       (reference "IN-12A_1") (unit 1) (value "IN-12A DAUGHTER") (footprint "nixie_tube_clock:nixie_daughter")
@@
     )
     (path "/bd472f43-1e2b-4c52-8cb4-5e5e311ab0b3/1ab12b00-7983-46e0-b147-9e396a057612"
-      (reference "TP1") (unit 1) (value "TestPoint") (footprint "TestPoint:TestPoint_Pad_D1.5mm")
+      (reference "TP1") (unit 1) (value "TestPoint") (footprint "TestPoint:TestPoint_Pad_D3.0mm")
     )
     (path "/bd472f43-1e2b-4c52-8cb4-5e5e311ab0b3/7fa92257-ada3-4736-852e-eb59d3a99b8e"
-      (reference "TP2") (unit 1) (value "TestPoint") (footprint "TestPoint:TestPoint_Pad_D1.5mm")
+      (reference "TP2") (unit 1) (value "TestPoint") (footprint "TestPoint:TestPoint_Pad_D3.0mm")
     )
     (path "/bd472f43-1e2b-4c52-8cb4-5e5e311ab0b3/47af5988-7854-4bcc-8c2e-1c19b8fa5f31"
-      (reference "TP3") (unit 1) (value "TestPoint") (footprint "TestPoint:TestPoint_Pad_D1.5mm")
+      (reference "TP3") (unit 1) (value "TestPoint") (footprint "TestPoint:TestPoint_Pad_D3.0mm")
     )
     (path "/bd472f43-1e2b-4c52-8cb4-5e5e311ab0b3/4ecea743-651a-4272-800a-6d7527db6c7f"
-      (reference "TP4") (unit 1) (value "TestPoint") (footprint "TestPoint:TestPoint_Pad_D1.5mm")
+      (reference "TP4") (unit 1) (value "TestPoint") (footprint "TestPoint:TestPoint_Pad_D3.0mm")
     )
     (path "/bd472f43-1e2b-4c52-8cb4-5e5e311ab0b3/32c66171-3f37-400d-8689-1e41d48dfdb8"
-      (reference "TP5") (unit 1) (value "TestPoint") (footprint "TestPoint:TestPoint_Keystone_5000-5004_Miniature")
+      (reference "TP5") (unit 1) (value "TestPoint") (footprint "TestPoint:TestPoint_Pad_D3.0mm")
     )
     (path "/bd472f43-1e2b-4c52-8cb4-5e5e311ab0b3/e02ff890-f4f8-4b28-b3ff-2c0b05e762d0"

Commit message: 1
Other:
- note added: "6-32 x 3/4 in MF standoff to front panel same for rear but FF"
Changed lines of the file:
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@@
+    (effects (font (size 1.27 1.27)) (justify left bottom))
+  )
+  (text "6-32 x 3/4 in MF standoff to front panel\nsame for rear but FF"
+    (at 29.21 16.51 0)
     (effects (font (size 1.27 1.27)) (justify left bottom))
   )

Commit message: fab stuff
Parts:
- added J? (x2): itsy bitsy sockets, symbol nixie-tube-clock:BOMTIE
- added PS?: VEL24US120-US-JA, symbol nixie-tube-clock:BOMTIE
Other:
- note removed: "x2 CES-114-01-T-S for itsy bitsy"
Changed lines of the file:
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@@
   )
   (text "wall brick P/N\nVEL24US120-US-JA\npos center\n2.1mmID 5.5mmOD 12mmL"
-    (at 29.21 34.29 0)
+    (at 25.4 27.305 0)
     (effects (font (size 1.27 1.27)) (justify left bottom))
   )
@@
   )
   (text "minute2" (at 240.03 118.11 0)
-    (effects (font (size 1.27 1.27)) (justify left bottom))
-  )
-  (text "x2 CES-114-01-T-S\n for itsy bitsy" (at 114.3 24.13 0)
     (effects (font (size 1.27 1.27)) (justify left bottom))
   )
@@
     (pin "1")
     (pin "2")
+  )
+  (symbol (lib_id "nixie-tube-clock:BOMTIE") (at 113.665 20.32 0) (unit 1)
+    (in_bom yes) (on_board yes) (fields_autoplaced)
+    (property "Reference" "J?" (id 0) (at 115.57 19.0499 0)
+      (effects (font (size 1.27 1.27)) (justify left))
+    )
+    (property "Value" "itsy bitsy sockets" (id 1) (at 115.57 21.5899 0)
+      (effects (font (size 1.27 1.27)) (justify left))
+    )
+    (property "Footprint" "" (id 2) (at 113.665 20.32 0)
+      (effects (font (size 1.27 1.27)) hide)
+    )
+    (property "Datasheet" "CES-114-01-T-S " (id 3) (at 113.665 20.32 0)
+      (effects (font (size 1.27 1.27)) hide)
+    )
   )
   (symbol (lib_id "Device:R_US") (at 104.14 62.23 90) (unit 1)
@@
     (pin "1")
   )
+  (symbol (lib_id "nixie-tube-clock:BOMTIE") (at 56.515 22.225 0) (unit 1)
+    (in_bom yes) (on_board yes) (fields_autoplaced)
+    (property "Reference" "PS?" (id 0) (at 58.42 20.9549 0)
+      (effects (font (size 1.27 1.27)) (justify left))
+    )
+    (property "Value" "VEL24US120-US-JA" (id 1) (at 58.42 23.4949 0)
+      (effects (font (size 1.27 1.27)) (justify left))
+    )
+    (property "Footprint" "" (id 2) (at 56.515 22.225 0)
+      (effects (font (size 1.27 1.27)) hide)
+    )
+    (property "Datasheet" "VEL24US120-US-JA" (id 3) (at 56.515 22.225 0)
+      (effects (font (size 1.27 1.27)) hide)
+    )
+  )
   (symbol (lib_id "power:+5V") (at 162.56 34.29 0) (mirror y) (unit 1)
     (in_bom yes) (on_board yes) (fields_autoplaced)
@@
     )
     (pin "1")
+  )
+  (symbol (lib_id "nixie-tube-clock:BOMTIE") (at 113.665 15.875 0) (unit 1)
+    (in_bom yes) (on_board yes) (fields_autoplaced)
+    (property "Reference" "J?" (id 0) (at 115.57 14.6049 0)
+      (effects (font (size 1.27 1.27)) (justify left))
+    )
+    (property "Value" "itsy bitsy sockets" (id 1) (at 115.57 17.1449 0)
+      (effects (font (size 1.27 1.27)) (justify left))
+    )
+    (property "Footprint" "" (id 2) (at 113.665 15.875 0)
+      (effects (font (size 1.27 1.27)) hide)
+    )
+    (property "Datasheet" "CES-114-01-T-S " (id 3) (at 113.665 15.875 0)
+      (effects (font (size 1.27 1.27)) hide)
+    )
   )
   (symbol (lib_id "Device:R_US") (at 149.86 151.13 0) (unit 1)
@@
     (path "/707afb61-7651-44ce-83e2-006ac05910c6" (page "2"))
     (path "/0f164f5f-ce46-4a0f-aed4-90543affee8b" (page "3"))
+    (path "/f5443302-197b-472a-b14a-60a9f67d3b3f" (page "7"))
     (path "/34ce4e81-1933-462b-a9be-0bc1cc3bfb0e" (page "4"))
     (path "/6b34c966-1922-4f1d-a19b-a364558218be" (page "5"))
     (path "/b60e71a5-a78e-4615-99b1-d6b13e2875f1" (page "6"))
-    (path "/f5443302-197b-472a-b14a-60a9f67d3b3f" (page "7"))
     (path "/8a841f68-6f4f-41f7-ae0b-0bd43ab5ff74" (page "8"))
   )
@@
       (reference "J5") (unit 1) (value "LPPB121NFSC-RC") (footprint "")
     )
+    (path "/4036c7e1-44ef-4ba7-9d7f-ec3363fce416"
+      (reference "J?") (unit 1) (value "itsy bitsy sockets") (footprint "")
+    )
+    (path "/e397848a-7c5f-4dca-a1cb-8dda896b045e"
+      (reference "J?") (unit 1) (value "itsy bitsy sockets") (footprint "")
+    )
     (path "/bd472f43-1e2b-4c52-8cb4-5e5e311ab0b3/037a1ddf-0d76-445c-a0df-c95c82634474"
       (reference "L1") (unit 1) (value "1mH") (footprint "nixie_tube_clock:PM2120")
     )
+    (path "/adeb541d-0e55-423b-b1a5-ac8cec777f8d"
+      (reference "PS?") (unit 1) (value "VEL24US120-US-JA") (footprint "")
+    )
     (path "/bd472f43-1e2b-4c52-8cb4-5e5e311ab0b3/b0597cd8-4a0a-4aa4-8f24-2a7e34f3151b"
