File: nixie-tube-clock-hw/nixie_daughter/nixie_daughter.kicad_pcb (KiCad board)
At the start: 2 copper layers, 28 x 44 mm, 4 parts, among them J1 HPH1-A-12-UA

Commit message: 1
Parts:
- renumbered IN-12B to IN-12
Changed lines of the file:
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@@
       (outputformat 1)
       (mirror false)
-      (drillshape 1)
+      (drillshape 0)
       (scaleselection 1)
-      (outputdirectory "")
+      (outputdirectory "fab/")
     )
   )
@@
     (property "Sheetname" "")
     (attr through_hole)
-    (fp_text reference "IN-12B" (at 0 19 unlocked) (layer "F.SilkS")
+    (fp_text reference "IN-12" (at 0.000008 18.999988 unlocked) (layer "F.SilkS")
       (effects (font (size 2 2) (thickness 0.3) italic))
     )
@@
     (pts (xy 109 132) (xy 137 132))
     (height 14)
-    (gr_text "28.0000 mm" (at 123 144.2) (layer "Dwgs.User")
+    (gr_text "1102.3622 mils" (at 123 144.2) (layer "Dwgs.User")
       (effects (font (size 1.5 1.5) (thickness 0.3)))
     )
@@
     (pts (xy 113 92) (xy 113 136))
     (height 16)
-    (gr_text "44.0000 mm" (at 95.2 114 90) (layer "Dwgs.User")
+    (gr_text "1732.2835 mils" (at 95.2 114 90) (layer "Dwgs.User")
       (effects (font (size 1.5 1.5) (thickness 0.3)))
     )
@@
     (pts (xy 123 114) (xy 123 132))
     (height 20)
-    (gr_text "18.0000 mm" (at 101.2 123 90) (layer "Dwgs.User")
+    (gr_text "708.6614 mils" (at 101.2 123 90) (layer "Dwgs.User")
       (effects (font (size 1.5 1.5) (thickness 0.3)))
     )
@@
     (pts (xy 123 114) (xy 123 95))
     (height -20)
-    (gr_text "19.0000 mm" (at 101.2 104.5 90) (layer "Dwgs.User")
+    (gr_text "748.0315 mils" (at 101.2 104.5 90) (layer "Dwgs.User")
       (effects (font (size 1.5 1.5) (thickness 0.3)))
     )
@@
     (pts (xy 113 132) (xy 133 132))
     (height 8)
-    (gr_text "20.0000 mm" (at 123 138.2) (layer "Dwgs.User")
-      (effects (font (size 1.5 1.5) (thickness 0.3)))
-    )
+    (gr_text "787.4016 mils" (at 123 138.2) (layer "Dwgs.User")
+      (effects (font (size 1.5 1.5) (thickness 0.3)))
+    )

Commit message: minor board / part changes
Routing:
- net Net-(IN-12B1-Pad4): track 16.9 -> 66.0 mm
- net Net-(IN-12B1-Pad11): track 33.0 -> 55.3 mm
- net Net-(IN-12B1-Pad1): track 32.8 -> 52.5 mm, vias 0 -> 2
- net Net-(IN-12B1-Pad6): track 10.0 -> 26.7 mm
- net Net-(IN-12B1-Pad10): track 26.5 -> 41.9 mm
- net Net-(IN-12B1-Pad5): track 13.3 -> 27.7 mm
- net Net-(IN-12B1-Pad9): track 22.5 -> 34.3 mm
- net Net-(IN-12B1-Pad3): track 22.5 -> 32.2 mm, vias 0 -> 1
- net Net-(IN-12B1-Pad2): track 28.1 -> 36.0 mm, vias 0 -> 1
- net Net-(IN-12B1-Pad8): track 16.9 -> 24.7 mm
- net Net-(IN-12B1-Pad7): track 12.1 -> 14.4 mm
- net Net-(IN-12B1-Pad12): track 41.5 -> 40.9 mm
